File: digital_signal_24V_to_5V.kicad_sch (KiCad schematic)
At the start: 5 parts, among them U2 4N35

Commit message: ready to upload
Parts:
- removed R2: 100k Ω, Resistor_THT:R_Axial_DIN0207_L6.3mm_D2.5mm_P2.54mm_Vertical, symbol Device:R
- R1, R3, R4: footprint Resistor_THT:R_Axial_DIN0207_L6.3mm_D2.5mm_P2.54mm_Vertical -> Resistor_SMD:R_0805_2012Metric
Connections:
- net GND: now also U2.6
Other:
- company: (none) -> ${company}
- title: (none) -> ${project_title} - ${board_title}
Changed lines of the file:
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@@
 (kicad_sch (version 20211123) (generator eeschema)
   (paper "A4")
+  (title_block
+    (title "${project_title} - ${board_title}")
+    (date "2022-08-11")
+    (rev "${git_describe}")
+    (company "${company}")
+    (comment 1 "${drawn_by}")
+    (comment 4 "${git_url}")
+  )
   (junction (at 148.59 93.345) (diameter 0) (color 0 0 0 0)
   )
   (junction (at 175.26 93.345) (diameter 0) (color 0 0 0 0)
-  )
-  (wire (pts (xy 167.64 74.295) (xy 175.26 74.295))
-    (stroke (width 0) (type default) (color 0 0 0 0))
-  )
-  (wire (pts (xy 148.59 74.295) (xy 160.02 74.295))
-    (stroke (width 0) (type default) (color 0 0 0 0))
   )
   (wire (pts (xy 181.61 84.455) (xy 181.61 64.135))
@@
   )
   (wire (pts (xy 148.59 100.965) (xy 215.9 100.965))
+    (stroke (width 0) (type default) (color 0 0 0 0))
+  )
+  (wire (pts (xy 148.59 76.835) (xy 175.26 76.835))
     (stroke (width 0) (type default) (color 0 0 0 0))
   )
@@
     (stroke (width 0) (type default) (color 0 0 0 0))
   )
-  (wire (pts (xy 175.26 93.345) (xy 175.26 74.295))
+  (wire (pts (xy 175.26 93.345) (xy 175.26 76.835))
     (stroke (width 0) (type default) (color 0 0 0 0))
   )
@@
     (stroke (width 0) (type default) (color 0 0 0 0))
   )
-  (wire (pts (xy 148.59 81.915) (xy 148.59 74.295))
+  (wire (pts (xy 148.59 81.915) (xy 148.59 76.835))
     (stroke (width 0) (type default) (color 0 0 0 0))
   )
@@
   (hierarchical_label "24-signal" (shape input) (at 91.44 81.915 180)
     (effects (font (size 1.27 1.27)) (justify right))
-  )
-  (symbol (lib_id "Device:R") (at 163.83 74.295 270) (mirror x) (unit 1)
-    (in_bom yes) (on_board yes)
-    (property "Reference" "R2" (id 0) (at 162.56 71.755 90)
-      (effects (font (size 1.27 1.27)) (justify left))
-    )
-    (property "Value" "100k Ω" (id 1) (at 160.02 78.105 90)
-      (effects (font (size 1.27 1.27)) (justify left))
-    )
-    (property "Footprint" "Resistor_THT:R_Axial_DIN0207_L6.3mm_D2.5mm_P2.54mm_Vertical" (id 2) (at 163.83 76.073 90)
-      (effects (font (size 1.27 1.27)) hide)
-    )
-    (property "Datasheet" "~" (id 3) (at 163.83 74.295 0)
-      (effects (font (size 1.27 1.27)) hide)
-    )
-    (pin "1")
-    (pin "2")
   )
   (symbol (lib_id "power:+5V") (at 181.61 64.135 0) (mirror y) (unit 1)
@@
       (effects (font (size 1.27 1.27)) (justify left))
     )
-    (property "Footprint" "Resistor_THT:R_Axial_DIN0207_L6.3mm_D2.5mm_P2.54mm_Vertical" (id 2) (at 163.83 95.123 90)
+    (property "Footprint" "Resistor_SMD:R_0805_2012Metric" (id 2) (at 163.83 95.123 90)
       (effects (font (size 1.27 1.27)) hide)
     )
@@
       (effects (font (size 1.27 1.27)) (justify left))
     )
-    (property "Footprint" "Resistor_THT:R_Axial_DIN0207_L6.3mm_D2.5mm_P2.54mm_Vertical" (id 2) (at 120.65 80.137 90)
+    (property "Footprint" "Resistor_SMD:R_0805_2012Metric" (id 2) (at 120.65 80.137 90)
       (effects (font (size 1.27 1.27)) hide)
     )
@@
       (effects (font (size 1.27 1.27)) (justify left))
     )
-    (property "Footprint" "Resistor_THT:R_Axial_DIN0207_L6.3mm_D2.5mm_P2.54mm_Vertical" (id 2) (at 163.83 86.233 90)
+    (property "Footprint" "Resistor_SMD:R_0805_2012Metric" (id 2) (at 163.83 86.233 90)
       (effects (font (size 1.27 1.27)) hide)
     )
