File: digital_signal_24V_to_5V_breakout.kicad_sch (KiCad schematic)
At the start: 3 parts, among them J1 Conn_01x04_Male, J2 Conn_01x04_Female, U1 R-785.0-0.5

Commit message: ready to upload
Parts:
- removed U1: R-785.0-0.5, Converter_DCDC:Converter_DCDC_RECOM_R-78E-0.5_THT, symbol Regulator_Switching:R-785.0-0.5
- added H1, H2: MountingHole, MountingHole:MountingHole_3.2mm_M3, symbol Mechanical:MountingHole
- added U1: LM22676MR-ADJ/NOPB, Package_SO:Texas_HSOP-8-1EP_3.9x4.9mm_P1.27mm_ThermalVias, symbol LM22676MR-ADJ_NOPB:LM22676MR-ADJ{brace}slash}NOPB
- J1, J2: footprint (none) -> Connector_Molex:Molex_Micro-Fit_3.0_43045-0400_2x02_P3.00mm_Horizontal
Connections:
- net +24V: now also J2.2 (Pin_2), U1.7 (VIN); no longer J1.3 (Pin_3)
- net +5V: now also J1.2 (Pin_2), U1.8 (SW); no longer J2.3 (Pin_3)
- net GND: now also J1.1 (Pin_1), J2.1 (Pin_1), U1.5 (EN), U1.6 (GND), U1.9 (EPAD); no longer J1.4 (Pin_4), J2.4 (Pin_4)
- net Signal A 24V: now also J2.4 (Pin_4); no longer J1.1 (Pin_1)
- net Signal A 5V: now also J1.4 (Pin_4); no longer J2.1 (Pin_1)
- net Signal B 24V: now also J2.3 (Pin_3); no longer J1.2 (Pin_2)
- net Signal B 5V: now also J1.3 (Pin_3); no longer J2.2 (Pin_2)
- no-connect marks 0 -> 2
Other:
- company: (none) -> ${company}
- title: (none) -> ${project_title} - ${board_title}
- moved on the sheet: J1, J2
